Commit message: Added crisp/ directory and instructions how to setup crisp_gym. Modified PS5 teleop node to accept --crisp-teleop argument which makes the node compatible with CRISP teleoperation

File: src/franka_fm_gazebo/urdf/rgb_camera.xacro (robot description, xacro)
@@ -57,5 +57,5 @@
       <!-- rotate into optical frame (z forward, x right, y down),
            problem is that camera is spawned so that it points along x axis -->
-      <origin xyz="0 0 0" rpy="${pi} -${pi} -${pi/2}" />
+      <origin xyz="0 0 0" rpy="${pi} -${pi} -${pi}" />
     </joint>
     <!-- Gazebo sensor -->
